File: SmartThermo1.4.brd (EAGLE design)
At the start: 100 x 80 mm, 26 parts, among them IC1 LM35DT, J1 AVR_SPI_PRG_6NS, J3 POWER_JACKPTH, P1 10K, Q1 IRF7509, Q2 IRF7509, U1 ATMEGA328P_PDIP, U2 LCD-16X2NOHOLES

Commit message: Add files via upload
Parts:
- moved FAN 3.81 mm to (90.2, 33.0)
- moved HEAT_ELMNT 3.81 mm to (90.2, 45.7)
Routing:
- net GND: track 0.00 -> 276.3 mm
- net +5V: track 0.00 -> 270.4 mm
- net N$1: track 0.00 -> 119.1 mm
- net N$17: track 0.00 -> 65.9 mm
- net N$6: track 0.00 -> 56.9 mm
- net N$3: track 0.00 -> 42.9 mm
- net N$10: track 0.00 -> 41.6 mm
- net N$5: track 0.00 -> 41.3 mm
- net N$11: track 0.00 -> 41.2 mm
- net N$9: track 0.00 -> 41.2 mm
- net N$7: track 0.00 -> 41.2 mm
- net N$8: track 0.00 -> 37.1 mm
- net N$13: track 0.00 -> 35.9 mm
- net N$19: track 0.00 -> 25.8 mm
- net N$12: track 0.00 -> 24.9 mm
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