File: SmartThermo1.9.brd (EAGLE design)
At the start: 100 x 80 mm, 32 parts, among them J1 AVR_SPI_PRG_6NS, J3 POWER_JACKPTH, P1 10K, Q1 IRF7509, Q2 IRF7509, U1 ATMEGA328P_PDIP, U2 LCD-16X2NOHOLES

Commit message: Add files via upload
Parts:
- moved H1 1.61 mm to (94.7, 4.83)
- moved H4 0.25 mm to (95.2, 75.2)
Other:
- outline, holes or cut-outs redrawn
- board text added: "Temperature Control Board"
- board text added: "Version 1.0"
Changed lines of the file:
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@@
 <wire x1="0" y1="0" x2="100.0052" y2="0" width="0" layer="20"/>
 <wire x1="100.0052" y1="0" x2="100.0052" y2="79.9848" width="0" layer="20"/>
-<wire x1="100.0052" y1="79.9848" x2="0" y2="79.68" width="0" layer="20"/>
-<wire x1="0" y1="79.68" x2="0" y2="0" width="0" layer="20"/>
-<text x="15.24" y="74.93" size="1.778" layer="21">Group 9</text>
+<wire x1="100.0052" y1="79.9848" x2="0" y2="79.9848" width="0" layer="20"/>
+<wire x1="0" y1="79.9848" x2="0" y2="0" width="0" layer="20"/>
+<text x="68.834" y="74.168" size="1.778" layer="21" rot="R180">Group 9</text>
+<text x="60.198" y="68.326" size="1.778" layer="21">Version 1.0</text>
+<text x="59.944" y="76.708" size="1.778" layer="21">Temperature Control Board</text>
 </plain>
 <attributes>
@@
 </element>
 <element name="FAN" library="pinhead" library_urn="urn:adsk.eagle:library:325" package="1X02/90" package3d_urn="urn:adsk.eagle:package:22437/1" value="" x="3.81" y="60.96" rot="R90"/>
-<element name="H1" library="holes" library_urn="urn:adsk.eagle:library:237" package="3,0" package3d_urn="urn:adsk.eagle:package:14277/1" value="MOUNT-HOLE3.0" x="95.25" y="6.35"/>
+<element name="H1" library="holes" library_urn="urn:adsk.eagle:library:237" package="3,0" package3d_urn="urn:adsk.eagle:package:14277/1" value="MOUNT-HOLE3.0" x="94.742" y="4.826"/>
 <element name="H2" library="holes" library_urn="urn:adsk.eagle:library:237" package="3,0" package3d_urn="urn:adsk.eagle:package:14277/1" value="MOUNT-HOLE3.0" x="5.08" y="5.08"/>
 <element name="H3" library="holes" library_urn="urn:adsk.eagle:library:237" package="3,0" package3d_urn="urn:adsk.eagle:package:14277/1" value="MOUNT-HOLE3.0" x="5.08" y="74.93"/>
-<element name="H4" library="holes" library_urn="urn:adsk.eagle:library:237" package="3,0" package3d_urn="urn:adsk.eagle:package:14277/1" value="MOUNT-HOLE3.0" x="95.25" y="74.93"/>
+<element name="H4" library="holes" library_urn="urn:adsk.eagle:library:237" package="3,0" package3d_urn="urn:adsk.eagle:package:14277/1" value="MOUNT-HOLE3.0" x="95.25" y="75.184"/>
 <element name="HEAT_ELMNT" library="pinhead" library_urn="urn:adsk.eagle:library:325" package="1X02/90" package3d_urn="urn:adsk.eagle:package:22437/1" value="" x="3.81" y="44.45" rot="R90"/>
 <element name="J1" library="SparkFun-Connectors" package="2X3-NS" value="AVR_SPI_PRG_6NS" x="67.31" y="24.13" rot="R180"/>
@@
 <wire x1="23.252953125" y1="53.0127875" x2="26.96" y2="52.365" width="0.254" layer="1"/>
 <wire x1="26.96" y1="52.365" x2="20.32" y2="47.498" width="0.254" layer="1"/>
-<wire x1="20.32" y1="47.498" x2="11.176" y2="47.498" width="0.254" layer="1"/>
-<wire x1="11.176" y1="47.498" x2="8.636" y2="38.354" width="0.254" layer="1"/>
-<wire x1="8.636" y1="38.354" x2="8.726290625" y2="42.086" width="0.254" layer="1"/>
+<wire x1="20.32" y1="47.498" x2="10.922" y2="47.498" width="0.254" layer="1"/>
+<wire x1="10.922" y1="47.498" x2="8.89" y2="38.608" width="0.254" layer="1"/>
+<wire x1="8.89" y1="38.608" x2="8.726290625" y2="42.086" width="0.254" layer="1"/>
 <wire x1="8.726290625" y1="42.086" x2="8.83515" y2="42.086" width="0.254" layer="1"/>
 <wire x1="8.83515" y1="42.086" x2="9.476" y2="42.72685" width="0.254" layer="1"/>
 <wire x1="9.476" y1="42.72685" x2="9.476" y2="43.63315" width="0.254" layer="1"/>
-<wire x1="9.476" y1="43.63315" x2="8.83515" y2="44.274" width="0.254" layer="1"/>
+<wire x1="8.83515" y1="44.274" x2="9.476" y2="43.63315" width="0.254" layer="1"/>
 <wire x1="6.40485" y1="44.626" x2="5.764" y2="45.26685" width="0.254" layer="1"/>
 <wire x1="5.764" y1="45.26685" x2="5.764" y2="46.17315" width="0.254" layer="1"/>

Commit message: Add files via upload
Routing:
- net N$21: track 210.2 -> 199.7 mm
Changed lines of the file:
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@@
 <contactref element="D2" pad="A"/>
 <contactref element="D3" pad="K"/>
-<wire x1="23.252953125" y1="53.0127875" x2="17.78" y2="49.53" width="0.254" layer="1"/>
+<wire x1="22.95711875" y1="52.824528125" x2="23.252953125" y2="53.0127875" width="0.254" layer="1"/>
+<wire x1="22.95711875" y1="52.824528125" x2="17.78" y2="49.53" width="0.254" layer="1"/>
 <wire x1="23.252953125" y1="53.0127875" x2="23.368" y2="53.086" width="0.254" layer="1"/>
 <wire x1="23.368" y1="53.086" x2="26.96" y2="53.015" width="0.254" layer="1"/>
 <wire x1="23.252953125" y1="53.0127875" x2="26.96" y2="52.365" width="0.254" layer="1"/>
-<wire x1="26.96" y1="52.365" x2="20.32" y2="47.498" width="0.254" layer="1"/>
-<wire x1="20.32" y1="47.498" x2="10.922" y2="47.498" width="0.254" layer="1"/>
-<wire x1="10.922" y1="47.498" x2="8.89" y2="38.608" width="0.254" layer="1"/>
-<wire x1="8.89" y1="38.608" x2="8.726290625" y2="42.086" width="0.254" layer="1"/>
-<wire x1="8.726290625" y1="42.086" x2="8.83515" y2="42.086" width="0.254" layer="1"/>
-<wire x1="8.83515" y1="42.086" x2="9.476" y2="42.72685" width="0.254" layer="1"/>
-<wire x1="9.476" y1="42.72685" x2="9.476" y2="43.63315" width="0.254" layer="1"/>
-<wire x1="8.83515" y1="44.274" x2="9.476" y2="43.63315" width="0.254" layer="1"/>
-<wire x1="6.40485" y1="44.626" x2="5.764" y2="45.26685" width="0.254" layer="1"/>
-<wire x1="5.764" y1="45.26685" x2="5.764" y2="46.17315" width="0.254" layer="1"/>
 <wire x1="9.476" y1="59.23685" x2="9.476" y2="60.14315" width="0.254" layer="1"/>
 <wire x1="9.476" y1="60.14315" x2="9.170546875" y2="60.448603125" width="0.254" layer="1"/>
@@
 <wire x1="9.230546875" y1="62.928603125" x2="23.671" y2="62.928603125" width="0.254" layer="1"/>
 <wire x1="23.671" y1="62.928603125" x2="23.671" y2="58.483875" width="0.254" layer="1"/>
-<wire x1="8.83515" y1="44.274" x2="8.843665625" y2="44.626" width="0.254" layer="1"/>
-<wire x1="5.764" y1="46.17315" x2="5.9958625" y2="55.7567125" width="0.254" layer="1"/>
-<wire x1="8.843665625" y1="44.626" x2="6.40485" y2="44.626" width="0.254" layer="1"/>
 <wire x1="5.9958625" y1="55.7567125" x2="9.476" y2="59.23685" width="0.254" layer="1"/>
 <wire x1="34.988125" y1="58.723" x2="38.562" y2="62.296875" width="0.254" layer="1"/>
@@
 <wire x1="35.306" y1="46.482" x2="35.306" y2="44.196" width="0.254" layer="1"/>
 <wire x1="35.306" y1="44.196" x2="37.22" y2="44.45" width="0.254" layer="1"/>
+<wire x1="20.066" y1="47.244" x2="23.622" y2="50.038" width="0.254" layer="1"/>
+<wire x1="20.066" y1="47.244" x2="10.414" y2="47.244" width="0.254" layer="1"/>
+<wire x1="10.414" y1="47.244" x2="10.414" y2="44.45" width="0.254" layer="1"/>
+<wire x1="10.414" y1="44.45" x2="5.08" y2="44.45" width="0.254" layer="1"/>
+<wire x1="5.08" y1="44.45" x2="5.08" y2="54.356" width="0.254" layer="1"/>
+<wire x1="5.08" y1="54.356" x2="5.9958625" y2="55.7567125" width="0.254" layer="1"/>
+<wire x1="23.622" y1="50.038" x2="22.95711875" y2="52.824528125" width="0.254" layer="1"/>
 </signal>
 <signal name="N$26">
