File: SmartThermo1.9.brd (EAGLE design)
At the start: 100 x 80 mm, 32 parts, among them J1 AVR_SPI_PRG_6NS, J3 POWER_JACKPTH, P1 10K, Q1 IRF7509, Q2 IRF7509, U1 ATMEGA328P_PDIP, U2 LCD-16X2NOHOLES

Commit message: Add files via upload
Routing:
- net N$21: track 199.7 -> 167.8 mm
Changed lines of the file:
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@@
 <via x="27.94" y="2.54" extent="1-16" drill="0.35"/>
 <via x="60.96" y="49.53" extent="1-16" drill="0.35"/>
+<via x="33.02" y="61.976" extent="1-16" drill="0.35"/>
 </signal>
 <signal name="N$2">
@@
 <wire x1="8.83515" y1="63.324" x2="9.230546875" y2="62.928603125" width="0.254" layer="1"/>
 <wire x1="23.671" y1="58.483875" x2="23.939875" y2="58.215" width="0.254" layer="1"/>
-<wire x1="9.292346875" y1="65.483" x2="9.398" y2="69.85" width="0.254" layer="1"/>
+<wire x1="25.294346875" y1="65.229" x2="25.4" y2="69.596" width="0.254" layer="1"/>
 <wire x1="23.939875" y1="58.215" x2="29.146125" y2="58.215" width="0.254" layer="1"/>
 <wire x1="9.170546875" y1="60.448603125" x2="9.186971875" y2="61.1274875" width="0.254" layer="1"/>
@@
 <wire x1="38.562" y1="62.296875" x2="38.562" y2="64.13751875" width="0.254" layer="1"/>
 <wire x1="38.562" y1="64.13751875" x2="37.21651875" y2="65.483" width="0.254" layer="1"/>
-<wire x1="37.21651875" y1="65.483" x2="9.292346875" y2="65.483" width="0.254" layer="1"/>
-<wire x1="9.398" y1="69.85" x2="28.956" y2="70.104" width="0.254" layer="1"/>
+<wire x1="37.21651875" y1="65.483" x2="25.294346875" y2="65.229" width="0.254" layer="1"/>
+<wire x1="25.4" y1="69.596" x2="28.956" y2="70.104" width="0.254" layer="1"/>
 <wire x1="28.956" y1="70.104" x2="29.972" y2="68.58" width="0.254" layer="1"/>
 <wire x1="29.972" y1="68.58" x2="40.132" y2="67.818" width="0.254" layer="1"/>

Commit message: Add files via upload
Routing:
- net N$21: track 167.8 -> 31.4 mm, vias 0 -> 1
Changed lines of the file:
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@@
 <contactref element="D2" pad="A"/>
 <contactref element="D3" pad="K"/>
-<wire x1="22.95711875" y1="52.824528125" x2="23.252953125" y2="53.0127875" width="0.254" layer="1"/>
-<wire x1="22.95711875" y1="52.824528125" x2="17.78" y2="49.53" width="0.254" layer="1"/>
-<wire x1="23.252953125" y1="53.0127875" x2="23.368" y2="53.086" width="0.254" layer="1"/>
-<wire x1="23.368" y1="53.086" x2="26.96" y2="53.015" width="0.254" layer="1"/>
-<wire x1="23.252953125" y1="53.0127875" x2="26.96" y2="52.365" width="0.254" layer="1"/>
-<wire x1="9.476" y1="59.23685" x2="9.476" y2="60.14315" width="0.254" layer="1"/>
-<wire x1="9.476" y1="60.14315" x2="9.170546875" y2="60.448603125" width="0.254" layer="1"/>
-<wire x1="8.83515" y1="61.136" x2="6.40485" y2="61.136" width="0.254" layer="1"/>
-<wire x1="6.40485" y1="61.136" x2="5.764" y2="61.77685" width="0.254" layer="1"/>
-<wire x1="5.764" y1="61.77685" x2="5.764" y2="62.68315" width="0.254" layer="1"/>
-<wire x1="5.764" y1="62.68315" x2="6.40485" y2="63.324" width="0.254" layer="1"/>
-<wire x1="6.40485" y1="63.324" x2="8.83515" y2="63.324" width="0.254" layer="1"/>
-<wire x1="8.83515" y1="63.324" x2="9.230546875" y2="62.928603125" width="0.254" layer="1"/>
-<wire x1="23.671" y1="58.483875" x2="23.939875" y2="58.215" width="0.254" layer="1"/>
-<wire x1="25.294346875" y1="65.229" x2="25.4" y2="69.596" width="0.254" layer="1"/>
-<wire x1="23.939875" y1="58.215" x2="29.146125" y2="58.215" width="0.254" layer="1"/>
-<wire x1="9.170546875" y1="60.448603125" x2="9.186971875" y2="61.1274875" width="0.254" layer="1"/>
-<wire x1="9.186971875" y1="61.1274875" x2="8.83515" y2="61.136" width="0.254" layer="1"/>
-<wire x1="29.654125" y1="58.723" x2="34.988125" y2="58.723" width="0.254" layer="1"/>
-<wire x1="29.146125" y1="58.215" x2="29.654125" y2="58.723" width="0.254" layer="1"/>
-<wire x1="9.230546875" y1="62.928603125" x2="23.671" y2="62.928603125" width="0.254" layer="1"/>
-<wire x1="23.671" y1="62.928603125" x2="23.671" y2="58.483875" width="0.254" layer="1"/>
-<wire x1="5.9958625" y1="55.7567125" x2="9.476" y2="59.23685" width="0.254" layer="1"/>
-<wire x1="34.988125" y1="58.723" x2="38.562" y2="62.296875" width="0.254" layer="1"/>
-<wire x1="38.562" y1="62.296875" x2="38.562" y2="64.13751875" width="0.254" layer="1"/>
-<wire x1="38.562" y1="64.13751875" x2="37.21651875" y2="65.483" width="0.254" layer="1"/>
-<wire x1="37.21651875" y1="65.483" x2="25.294346875" y2="65.229" width="0.254" layer="1"/>
-<wire x1="25.4" y1="69.596" x2="28.956" y2="70.104" width="0.254" layer="1"/>
-<wire x1="28.956" y1="70.104" x2="29.972" y2="68.58" width="0.254" layer="1"/>
-<wire x1="29.972" y1="68.58" x2="40.132" y2="67.818" width="0.254" layer="1"/>
-<wire x1="40.132" y1="67.818" x2="40.132" y2="46.482" width="0.254" layer="1"/>
-<wire x1="40.132" y1="46.482" x2="35.306" y2="46.482" width="0.254" layer="1"/>
-<wire x1="35.306" y1="46.482" x2="35.306" y2="44.196" width="0.254" layer="1"/>
-<wire x1="35.306" y1="44.196" x2="37.22" y2="44.45" width="0.254" layer="1"/>
-<wire x1="20.066" y1="47.244" x2="23.622" y2="50.038" width="0.254" layer="1"/>
-<wire x1="20.066" y1="47.244" x2="10.414" y2="47.244" width="0.254" layer="1"/>
-<wire x1="10.414" y1="47.244" x2="10.414" y2="44.45" width="0.254" layer="1"/>
-<wire x1="10.414" y1="44.45" x2="5.08" y2="44.45" width="0.254" layer="1"/>
-<wire x1="5.08" y1="44.45" x2="5.08" y2="54.356" width="0.254" layer="1"/>
-<wire x1="5.08" y1="54.356" x2="5.9958625" y2="55.7567125" width="0.254" layer="1"/>
-<wire x1="23.622" y1="50.038" x2="22.95711875" y2="52.824528125" width="0.254" layer="1"/>
+<wire x1="26.96" y1="53.015" x2="26.96" y2="52.365" width="0.254" layer="1"/>
+<wire x1="26.96" y1="52.365" x2="20.615" y2="52.365" width="0.254" layer="1"/>
+<wire x1="20.615" y1="52.365" x2="17.78" y2="49.53" width="0.254" layer="1"/>
+<wire x1="37.22" y1="44.45" x2="35.306" y2="44.45" width="0.254" layer="1"/>
+<via x="34.29" y="45.466" extent="1-16" drill="0.35"/>
+<wire x1="34.29" y1="45.466" x2="17.78" y2="49.53" width="0.254" layer="16"/>
+<wire x1="35.306" y1="44.45" x2="34.29" y2="45.466" width="0.254" layer="1"/>
 </signal>
 <signal name="N$26">

Commit message: Add files via upload
Parts:
- moved H3 10.2 mm to (5.08, 85.1)
- moved H4 9.43 mm to (94.5, 84.6)
Other:
- board size 100 x 80 mm -> 100 x 90 mm
Changed lines of the file:
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@@
 <plain>
 <wire x1="0" y1="0" x2="100.0052" y2="0" width="0" layer="20"/>
-<wire x1="100.0052" y1="0" x2="100.0052" y2="79.9848" width="0" layer="20"/>
-<wire x1="100.0052" y1="79.9848" x2="0" y2="79.9848" width="0" layer="20"/>
-<wire x1="0" y1="79.9848" x2="0" y2="0" width="0" layer="20"/>
-<text x="68.834" y="74.168" size="1.778" layer="21" rot="R180">Group 9</text>
-<text x="60.198" y="68.326" size="1.778" layer="21">Version 1.0</text>
-<text x="59.944" y="76.708" size="1.778" layer="21">Temperature Control Board</text>
+<wire x1="100.0052" y1="0" x2="100.0052" y2="89.9924" width="0" layer="20"/>
+<wire x1="100.0052" y1="89.9924" x2="0" y2="89.9924" width="0" layer="20"/>
+<wire x1="0" y1="89.9924" x2="0" y2="0" width="0" layer="20"/>
+<text x="62.484" y="84.582" size="1.778" layer="21" rot="R180">Group 9</text>
+<text x="68.072" y="82.804" size="1.778" layer="21">Version 1.0</text>
+<text x="18.796" y="83.058" size="1.778" layer="21">Temperature Control Board</text>
 </plain>
 <attributes>
@@
 <element name="H1" library="holes" library_urn="urn:adsk.eagle:library:237" package="3,0" package3d_urn="urn:adsk.eagle:package:14277/1" value="MOUNT-HOLE3.0" x="94.742" y="4.826"/>
 <element name="H2" library="holes" library_urn="urn:adsk.eagle:library:237" package="3,0" package3d_urn="urn:adsk.eagle:package:14277/1" value="MOUNT-HOLE3.0" x="5.08" y="5.08"/>
-<element name="H3" library="holes" library_urn="urn:adsk.eagle:library:237" package="3,0" package3d_urn="urn:adsk.eagle:package:14277/1" value="MOUNT-HOLE3.0" x="5.08" y="74.93"/>
-<element name="H4" library="holes" library_urn="urn:adsk.eagle:library:237" package="3,0" package3d_urn="urn:adsk.eagle:package:14277/1" value="MOUNT-HOLE3.0" x="95.25" y="75.184"/>
+<element name="H3" library="holes" library_urn="urn:adsk.eagle:library:237" package="3,0" package3d_urn="urn:adsk.eagle:package:14277/1" value="MOUNT-HOLE3.0" x="5.08" y="85.09"/>
+<element name="H4" library="holes" library_urn="urn:adsk.eagle:library:237" package="3,0" package3d_urn="urn:adsk.eagle:package:14277/1" value="MOUNT-HOLE3.0" x="94.488" y="84.582"/>
 <element name="HEAT_ELMNT" library="pinhead" library_urn="urn:adsk.eagle:library:325" package="1X02/90" package3d_urn="urn:adsk.eagle:package:22437/1" value="" x="3.81" y="44.45" rot="R90"/>
 <element name="J1" library="SparkFun-Connectors" package="2X3-NS" value="AVR_SPI_PRG_6NS" x="67.31" y="24.13" rot="R180"/>
@@
 <polygon width="0.1524" layer="1">
 <vertex x="0" y="0"/>
-<vertex x="0" y="80.01"/>
-<vertex x="100.33" y="80.01"/>
+<vertex x="0.762" y="89.154"/>
+<vertex x="101.092" y="89.154"/>
 <vertex x="100.33" y="0"/>
 </polygon>
@@
 <vertex x="0" y="0"/>
 <vertex x="99.06" y="0"/>
-<vertex x="99.06" y="80.01"/>
-<vertex x="0" y="80.01"/>
+<vertex x="100.33" y="89.662"/>
+<vertex x="1.27" y="89.662"/>
 </polygon>
 <via x="72.39" y="66.04" extent="1-16" drill="0.35"/>
@@
 <via x="12.954" y="75.184" extent="1-16" drill="0.35"/>
 </signal>
+<signal name="N$33">
+<via x="37.338" y="76.2" extent="1-16" drill="0.35"/>
+</signal>
+<signal name="N$34">
+<via x="56.388" y="86.106" extent="1-16" drill="0.35"/>
+</signal>
+<signal name="N$35">
+<via x="69.088" y="79.502" extent="1-16" drill="0.35"/>
+</signal>
+<signal name="N$36">
+<via x="23.876" y="87.63" extent="1-16" drill="0.35"/>
+</signal>
+<signal name="N$37">
+<via x="24.384" y="78.486" extent="1-16" drill="0.35"/>
+</signal>
+<signal name="N$38">
+<via x="40.386" y="84.074" extent="1-16" drill="0.35"/>
+</signal>
+<signal name="N$39">
+<via x="86.36" y="82.55" extent="1-16" drill="0.35"/>
+</signal>
+<signal name="N$40">
+<via x="93.98" y="73.66" extent="1-16" drill="0.35"/>
+</signal>
+<signal name="N$41">
+<via x="13.716" y="85.598" extent="1-16" drill="0.35"/>
+</signal>
 </signals>

Commit message: Add files via upload
Connections:
- net N$5: now also U1.4; no longer U1.3
Changed lines of the file:
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@@
 <signal name="N$5">
 <contactref element="U2" pad="4"/>
-<contactref element="U1" pad="3"/>
 <wire x1="28.702" y1="11.43" x2="28.702" y2="12.446" width="0.254" layer="16"/>
 <wire x1="25.4" y1="8.128" x2="28.702" y2="11.43" width="0.254" layer="16"/>
@@
 <wire x1="40.132" y1="33.528" x2="40.132" y2="23.876" width="0.254" layer="16"/>
 <wire x1="47.752" y1="41.148" x2="40.132" y2="33.528" width="0.254" layer="16"/>
-<wire x1="47.752" y1="45.212" x2="47.752" y2="41.148" width="0.254" layer="16"/>
-<wire x1="49.53" y1="46.99" x2="47.752" y2="45.212" width="0.254" layer="16"/>
+<wire x1="47.752" y1="41.148" x2="47.752" y2="45.212" width="0.254" layer="16"/>
+<contactref element="U1" pad="4"/>
+<wire x1="47.752" y1="45.212" x2="48.768" y2="45.212" width="0.1524" layer="16"/>
+<wire x1="48.768" y1="45.212" x2="49.53" y2="44.45" width="0.1524" layer="16"/>
 </signal>
 <signal name="N$7">
