File: SmartThermo1.9.sch (EAGLE design)
At the start: 32 parts, among them J1 AVR_SPI_PRG_6NS, J3 POWER_JACKPTH, P1 10K, Q1 IRF7509, Q2 IRF7509, U1 ATMEGA328P_PDIP, U2 LCD-16X2NOHOLES

Commit message: Add files via upload
Connections:
- net N$5: now also U1.PD2(INT0); no longer U1.PD1(TXD)
Changed lines of the file:
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@@
 <segment>
 <pinref part="U2" gate="G$1" pin="RS"/>
-<wire x1="152.4" y1="101.6" x2="152.4" y2="30.48" width="0.1524" layer="91"/>
-<pinref part="U1" gate="G$1" pin="PD1(TXD)"/>
-<wire x1="152.4" y1="30.48" x2="116.84" y2="30.48" width="0.1524" layer="91"/>
+<wire x1="152.4" y1="101.6" x2="152.4" y2="27.94" width="0.1524" layer="91"/>
+<pinref part="U1" gate="G$1" pin="PD2(INT0)"/>
+<wire x1="116.84" y1="27.94" x2="152.4" y2="27.94" width="0.1524" layer="91"/>
 </segment>
 </net>
